File: remote-camera.sch (EAGLE design)
At the start: 14 parts, among them Q1 IRF

Commit message: update
Parts:
- removed JP1: (no value), SparkFun:M023.5MM
- removed JP2: (no value), SparkFun:M03JST-PTH
- removed JP4: (no value), SparkFun:M03SCREW
- removed JP8: (no value), SparkFun:M02JST-PTH-2
- added C3: 0.1µ, resistor:C-EU025-024X044
Connections:
- removed net CONTROL: JP2.3, JP4.3, Q1.G, R1.2
- removed net HIGH-CURRENT: JP1.1, JP8.1, Q1.D
- new net N$2: C3.1, Q1.S
- net D3: now also Q1.G, R1.2
- net GND: now also C3.2, X1.4; no longer JP2.2, JP4.2, Q1.S
- net VCC: no longer JP1.2, JP2.1, JP4.1, JP8.2
- net VIN_MOTEINO: now also Q1.D, X1.1
Other:
- note removed: "CC-BY-SA 4.0"
- note removed: "PowerShield R2"
- note removed: "author: Felix Rusu"
- note removed: "http://lowpowerlab.com/powershield"
- moved on the sheet: X1
